File: euro-project-sensors-pcb/euro-project-sensors-pcb.kicad_pcb (KiCad board)
At the start: 2 copper layers, 25 parts, among them J1 CH0, J2 CH0, J3 CH0, J4 CH0

Commit message: dfgbdfbdb
Parts:
- added J10: CH1, Connector_RJ:RJ45_OST_PJ012-8P8CX_Vertical, F.Cu at (199.4, 116.8)
- added J11: CH2, Connector_PinHeader_2.54mm:PinHeader_1x04_P2.54mm_Vertical, F.Cu at (174.0, 87.6)
- added J12: CH2, Connector_PinHeader_2.54mm:PinHeader_1x04_P2.54mm_Vertical, F.Cu at (174.0, 83.8)
- added J13: CH2, Connector_PinHeader_2.54mm:PinHeader_1x04_P2.54mm_Vertical, F.Cu at (174.0, 80.0)
- added J14: CH2, Connector_RJ:RJ45_OST_PJ012-8P8CX_Vertical, F.Cu at (190.5, 74.9)
- added J15: CH2, Connector_RJ:RJ45_OST_PJ012-8P8CX_Vertical, F.Cu at (208.3, 74.9)
- added J16: CH3, Connector_PinHeader_2.54mm:PinHeader_1x04_P2.54mm_Vertical, F.Cu at (174.0, 44.5)
- added J17: CH3, Connector_PinHeader_2.54mm:PinHeader_1x04_P2.54mm_Vertical, F.Cu at (174.0, 48.3)
- added J18: CH3, Connector_PinHeader_2.54mm:PinHeader_1x04_P2.54mm_Vertical, F.Cu at (174.0, 52.1)
- added J19: CH3, Connector_RJ:RJ45_OST_PJ012-8P8CX_Vertical, F.Cu at (217.2, 57.1)
- added J20: CH3, Connector_RJ:RJ45_OST_PJ012-8P8CX_Vertical, F.Cu at (199.4, 57.1)
- added J21: CH4, Connector_PinHeader_2.54mm:PinHeader_1x04_P2.54mm_Vertical, F.Cu at (111.8, 147.3)
- added J22: CH4, Connector_PinHeader_2.54mm:PinHeader_1x04_P2.54mm_Vertical, F.Cu at (111.8, 143.5)
- added J23: CH4, Connector_PinHeader_2.54mm:PinHeader_1x04_P2.54mm_Vertical, F.Cu at (111.8, 139.7)
- added J24: CH5, Connector_PinHeader_2.54mm:PinHeader_1x04_P2.54mm_Vertical, F.Cu at (110.5, 111.8)
- added J25: CH1, Connector_PinHeader_2.54mm:PinHeader_1x04_P2.54mm_Vertical, F.Cu at (110.5, 108.0)
- added J26: CH1, Connector_PinHeader_2.54mm:PinHeader_1x04_P2.54mm_Vertical, F.Cu at (110.5, 104.1)
- added J27: CH6, Connector_PinHeader_2.54mm:PinHeader_1x04_P2.54mm_Vertical, F.Cu at (111.8, 87.6)
- added J28: CH6, Connector_PinHeader_2.54mm:PinHeader_1x04_P2.54mm_Vertical, F.Cu at (111.8, 83.8)
- added J29: CH6, Connector_PinHeader_2.54mm:PinHeader_1x04_P2.54mm_Vertical, F.Cu at (111.8, 80.0)
- added J30: CH7, Connector_PinHeader_2.54mm:PinHeader_1x04_P2.54mm_Vertical, F.Cu at (111.8, 52.1)
- added J31: CH7, Connector_PinHeader_2.54mm:PinHeader_1x04_P2.54mm_Vertical, F.Cu at (111.8, 48.3)
- added J32: CH7, Connector_PinHeader_2.54mm:PinHeader_1x04_P2.54mm_Vertical, F.Cu at (111.8, 44.5)
- added J33: CH5, Connector_RJ:RJ45_OST_PJ012-8P8CX_Vertical, F.Cu at (83.8, 116.8)
- added J34: CH5, Connector_RJ:RJ45_OST_PJ012-8P8CX_Vertical, F.Cu at (101.6, 116.8)
- added J35: CH6, Connector_RJ:RJ45_OST_PJ012-8P8CX_Vertical, F.Cu at (76.2, 74.9)
- added J36: CH6, Connector_RJ:RJ45_OST_PJ012-8P8CX_Vertical, F.Cu at (94.0, 74.9)
- added J37: CH7, Connector_RJ:RJ45_OST_PJ012-8P8CX_Vertical, F.Cu at (85.1, 57.1)
- added J38: CH7, Connector_RJ:RJ45_OST_PJ012-8P8CX_Vertical, F.Cu at (102.9, 57.1)
- added J39: CH4, Connector_RJ:RJ45_OST_PJ012-8P8CX_Vertical, F.Cu at (94.0, 134.6)
- added J40: CH4, Connector_RJ:RJ45_OST_PJ012-8P8CX_Vertical, F.Cu at (76.2, 134.6)
- added J5: CH0, Connector_PinHeader_2.54mm:PinHeader_1x04_P2.54mm_Vertical, F.Cu at (174.0, 139.1)
- added J6: CH1, Connector_PinHeader_2.54mm:PinHeader_1x04_P2.54mm_Vertical, F.Cu at (174.0, 104.1)
- added J7: CH1, Connector_PinHeader_2.54mm:PinHeader_1x04_P2.54mm_Vertical, F.Cu at (174.0, 111.8)
- added J8: CH1, Connector_PinHeader_2.54mm:PinHeader_1x04_P2.54mm_Vertical, F.Cu at (174.0, 108.0)
- added J9: CH1, Connector_RJ:RJ45_OST_PJ012-8P8CX_Vertical, F.Cu at (217.2, 116.8)
- added JP2: VCC-CH1, 000-jumpers-immo:SolderJumper-3-open-high-power, F.Cu at (177.8, 118.1)
- added JP3: VCC-CH2, 000-jumpers-immo:SolderJumper-3-open-high-power, F.Cu at (177.8, 73.7)
- added JP4: VCC-CH3, 000-jumpers-immo:SolderJumper-3-open-high-power, F.Cu at (177.8, 58.4)
- added JP5: VCC-CH5, 000-jumpers-immo:SolderJumper-3-open-high-power, F.Cu at (113.0, 118.1)
- added JP6: VCC-CH6, 000-jumpers-immo:SolderJumper-3-open-high-power, F.Cu at (114.3, 73.7)
- added JP7: VCC-CH7, 000-jumpers-immo:SolderJumper-3-open-high-power, F.Cu at (114.8, 59.2)
- added JP8: VCC_CH4, 000-jumpers-immo:SolderJumper-3-open-high-power, F.Cu at (113.0, 133.3)
- added REF**: MountingHole_3.2mm_M3_Pad_Via, MountingHole:MountingHole_3.2mm_M3_Pad_Via, F.Cu at (75.8, 125.7)
- added REF**: MountingHole_3.2mm_M3_Pad_Via, MountingHole:MountingHole_3.2mm_M3_Pad_Via, F.Cu at (217.2, 66.0)
- added REF**: MountingHole_3.2mm_M3_Pad_Via, MountingHole:MountingHole_3.2mm_M3_Pad_Via, F.Cu at (76.2, 66.0)
- added REF**: MountingHole_3.2mm_M3_Pad_Via, MountingHole:MountingHole_3.2mm_M3_Pad_Via, F.Cu at (217.2, 125.7)
- J2, J3: footprint Connector_PinHeader_1.27mm:PinHeader_1x04_P1.27mm_Vertical -> Connector_PinHeader_2.54mm:PinHeader_1x04_P2.54mm_Vertical
- JP1: value CH0-VCC-select -> VCC_CH0; footprint Jumper:SolderJumper-3_P1.3mm_Open_RoundedPad1.0x1.5mm_NumberLabels -> 000-jumpers-immo:SolderJumper-3-open-high-power
- moved J3 125.2 mm to (174.0, 142.9), turned to 90 degrees
- moved J4 116.1 mm to (190.5, 134.6), turned to 0 degrees
- moved J1 114.6 mm to (208.3, 134.6)
- moved JP1 95.6 mm to (177.8, 133.3), turned to 180 degrees
- moved A1 92.6 mm to (139.7, 108.0)
- moved A2 86.7 mm to (134.9, 78.7)
- moved J2 71.7 mm to (174.0, 146.7), turned to 90 degrees
- moved R14 51.8 mm to (168.6, 55.9)
- moved R13 51.5 mm to (168.6, 53.3)
- moved R12 51.2 mm to (168.6, 50.8)
- moved R11 51.0 mm to (168.6, 48.3)
- moved R10 50.7 mm to (168.6, 45.7)
- moved R18 38.2 mm to (168.6, 63.5)
- moved R16 36.7 mm to (168.6, 61.0)
- moved R15 36.5 mm to (168.6, 58.4)
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Routing:
- net /5V_BUS: track 0.00 -> 318.5 mm, vias 0 -> 2
- net /3V3_BUS: track 0.00 -> 250.3 mm, vias 0 -> 7
- net /SDA_CH4: track 0.00 -> 175.8 mm
- net /SDA_CH0: track 0.00 -> 167.6 mm
- net /SCL_CH4: track 0.00 -> 163.3 mm, vias 0 -> 1
- net /SCL_CH0: track 0.00 -> 157.8 mm
- net /SDA_CH5: track 0.00 -> 149.3 mm
- net /SCL_CH1: track 0.00 -> 129.9 mm
- net /SDA_CH1: track 0.00 -> 128.7 mm
- net /SDA_CH6: track 0.00 -> 125.4 mm
- net /SCL_CH5: track 0.00 -> 124.4 mm
- net /SDA_CH2: track 0.00 -> 115.4 mm
- net /SCL_CH2: track 0.00 -> 115.4 mm
- net /SCL_CH6: track 0.00 -> 108.6 mm
- net /SCL_CH3: track 0.00 -> 107.6 mm
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- added copper zone on B.Cu, net GND
- added copper zone on F.Cu, net GND
Other:
- board outline added: 153.7 x 109.2 mm
- board text added: "Channel: 0"
- board text added: "Channel: 1"
- board text added: "Channel: 2"
- board text added: "Channel: 3"
- board text added: "Channel: 4"
- board text added: "Channel: 5"
- board text added: "Channel: 6"
- board text added: "Channel: 7"
- board text added: "I2C - Mux"
- board text added: "PCB Design: Imogen Heard 27/10/23"
- board text added: "SCL"
- board text added: "SDA"
- board text added: "Sensors Expansion Board"
- board text added: "Vcc"
- board text added: "gnd"

Commit message: PCB design Revision
Parts:
- removed REF** (x4): MountingHole_3.2mm_M3_Pad_Via, MountingHole:MountingHole_3.2mm_M3_Pad_Via
- added C1: 100n, 000_Capacitors_Immo:C_0805_2012_HandSolder_kawaii, F.Cu at (138.4, 101.0)
- added C2: 100n, 000_Capacitors_Immo:C_0805_2012_HandSolder_kawaii, F.Cu at (118.7, 96.3)
- added EC1: 100u, Capacitor_SMD:CP_Elec_10x10, F.Cu at (134.4, 125.7)
- added EC2: 100u, Capacitor_SMD:CP_Elec_10x10, F.Cu at (167.2, 95.2)
- added H1: MountingHole, MountingHole:MountingHole_3.2mm_M3_Pad_Via, F.Cu at (76.2, 66.0)
- added H2: MountingHole, MountingHole:MountingHole_3.2mm_M3_Pad_Via, F.Cu at (217.2, 66.0)
- added H3: MountingHole, MountingHole:MountingHole_3.2mm_M3_Pad_Via, F.Cu at (76.2, 125.1)
- added H4: MountingHole, MountingHole:MountingHole_3.2mm_M3_Pad_Via, F.Cu at (217.2, 125.1)
- added J41: 7-24v In, TerminalBlock:TerminalBlock_Altech_AK300-2_P5.00mm, F.Cu at (132.8, 142.9)
- added U1: R-78C5.0-1.0, Converter_DCDC:Converter_DCDC_RECOM_R-78E-0.5_THT, F.Cu at (140.0, 112.3)
- added U2: AMS1117-3.3, Package_TO_SOT_SMD:SOT-223-3_TabPin2, F.Cu at (126.4, 95.2)
- moved A1 6.99 mm to (146.7, 108.0)
Routing:
- net /5V_BUS: track 318.5 -> 365.4 mm, vias 2 -> 4
- net /SDA_CH4: track 175.8 -> 212.2 mm, vias 0 -> 1
- net Net-(J41-Pin_2): track 0.00 -> 30.6 mm
- net GND: track 0.00 -> 18.1 mm, vias 0 -> 3
- net /3V3_BUS: track 250.3 -> 261.8 mm
- net /SCL: track 46.0 -> 52.9 mm
- net /SDA: track 43.0 -> 45.4 mm
- net /SDA_CH6: track 125.4 -> 123.4 mm
- net /VCC_CH6: track 54.3 -> 52.4 mm
- net /SCL_CH6: track 108.6 -> 106.8 mm
- net /VCC_CH4: track 64.8 -> 66.2 mm
- net /SCL_CH0: track 157.8 -> 158.9 mm
- net /VCC_CH1: track 49.0 -> 50.0 mm
- net /SCL_CH3: track 107.6 -> 108.6 mm
- net /SDA_CH3: track 87.7 -> 88.3 mm
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Other:
- board text added: "+5v"
- board text added: "+V"
- board text added: "Vin"
